File: ESP32-S3-Template.kicad_pcb (KiCad board)
At the start: 4 copper layers, 25.4 x 60 mm, 50 parts, among them J1 USB_TYPE_C_16PIN, J2 Conn_01x22, J3 Conn_01x22, Q1 S8050, Q2 S8050, Q3 FDC6330L, SW1 RESET, SW2 BOOT, U1 CH343P, U2 CH334F, U3 ESP32-S3-WROOM-1-N16R8, U5 XC6210B332MR, U6 USBLC6-2SC6, Y1 32.768kHz, Y2 12Mhz

Commit message: i think its ready for reddit.
Parts:
- FB1: value 500mA -> 1.5A; footprint Fuse:Fuse_0603_1608Metric -> Fuse:Fuse_1206_3216Metric
- R3: value 1k -> 5.1k
- moved C15 1.95 mm to (77.7, 120.4)
- moved C16 1.95 mm to (79.3, 120.4)
- moved C17 1.95 mm to (80.9, 120.4)
- moved FB1 1.12 mm to (82.9, 121.2)
Routing:
- net /ESP32-S3/VBUS: track 35.6 -> 28.1 mm, vias 5 -> 3
- net /ESP32-S3/3.3VUSB: track 46.5 -> 43.4 mm
- net GND: track 13.7 -> 11.5 mm, vias 23 -> 21
- net Net-(D1-K): track 1.54 -> 3.11 mm
- added copper zone on F.Cu, net /ESP32-S3/VBUS

Commit message: another full pass over the schematic and layout
Parts:
- moved C14 2.20 mm to (83.7, 113.8)
Routing:
- net GND: vias 21 -> 22

Commit message: pulled in brineomatic version
Parts:
- D2: renamed from D3; value LED -> RED
- R1: renamed from R11; value 100 -> 100R
- SW1, SW2: footprint Button_Switch_SMD:SW_SPST_B3U-1000P -> Button_Switch_THT:SW_Tactile_SPST_Angled_PTS645Vx58-2LFS
- U1: renamed from U3; footprint RF_Module:ESP32-S3-WROOM-1 -> yarrboard:ESP32-S3-WROOM-1
- U4: renamed from U2; footprint Package_DFN_QFN:QFN-24-1EP_4x4mm_P0.5mm_EP2.7x2.7mm_ThermalVias -> yarrboard:QFN-24-1EP_4x4mm_P0.5mm_EP2.7x2.7mm_ThermalVias
- U5: renamed from U1; footprint Package_DFN_QFN:QFN-16-1EP_3x3mm_P0.5mm_EP1.7x1.7mm_ThermalVias -> yarrboard:QFN-16-1EP_3x3mm_P0.5mm_EP1.7x1.7mm_ThermalVias
- renumbered C12 to C10, C5 to C11, C2 to C12, C4 to C13, C15 to C14, C16 to C15, C14 to C16, C10 to C18, C11 to C19, C3 to C2, C13 to C3, C8 to C4, C18 to C5, C9 to C8, C19 to C9, D2 to D3, J2 to J1, J3 to J2, J1 to J3, Q3 to Q1, Q1 to Q2, Q2 to Q3, R5 to R10, R4 to R11, R9 to R2, R10 to R3, R1 to R4, R2 to R5, R3 to R6, R8 to R7, R6 to R8, R7 to R9, U6 to U2, U5 to U3, Y2 to Y1, Y1 to Y2
Connections:
- D2 pad 1: GND -> Net-(D2-K)
- D2 pad 2: Net-(D3-A) -> +3.3V
- R6 pad 1: +3.3V -> Net-(D2-K)
- R6 pad 2: Net-(D3-A) -> GND
Routing:
- net Net-(D3-A): track 1.46 -> 0.00 mm
- net (no net): track 0.00 -> 1.46 mm
