File: esp32-s3.kicad_sch (KiCad schematic)
At the start: 47 parts, among them J1 USB_TYPE_C_16PIN, Q1 S8050, Q2 S8050, Q3 FDC6330L, SW1 RESET, SW2 BOOT, U1 CH343P, U2 CH334F, U3 ESP32-S3-WROOM-1-N16R8, U5 XC6210B332MR, U6 USBLC6-2SC6, Y1 32.768kHz, Y2 12Mhz

Commit message: board is fully routed.
Parts:
- U1: footprint Package_DFN_QFN:QFN-16-1EP_3x3mm_P0.5mm_EP1.7x1.7mm -> Package_DFN_QFN:QFN-16-1EP_3x3mm_P0.5mm_EP1.7x1.7mm_ThermalVias
- U2: footprint Package_DFN_QFN:QFN-24-1EP_4x4mm_P0.5mm_EP2.7x2.7mm -> Package_DFN_QFN:QFN-24-1EP_4x4mm_P0.5mm_EP2.7x2.7mm_ThermalVias
Connections:
- net ESP_USB+: now also U2.10 (D+2); no longer U2.12 (D+1)
- net ESP_USB-: now also U2.9 (D-2); no longer U2.11 (D-1)
- net UART_D+: now also U2.12 (D+1); no longer U2.10 (D+2)
- net UART_D-: now also U2.11 (D-1); no longer U2.9 (D-2)
- net GND renamed ESP_GND
Other:
- moved on the sheet: C18, Y2

Commit message: fully routed, erc+drc pass, 3d models
Parts:
- D2: value WS2812B-2020 -> WS2812B-Mini; footprint LED_SMD:LED_WS2812B-2020_PLCC4_2.0x2.0mm -> LED_SMD:LED_WS2812B-Mini_PLCC4_3.5x3.5mm; symbol LED:WS2812B-2020 -> LED:WS2812B; LCSC (none) -> C527089
- J1: symbol Connector:USB_C_Receptacle_USB2.0 -> Connector:USB_C_Receptacle_USB2.0_16P
- Q1, Q2: symbol Device:Q_NPN_BCE -> Transistor_BJT:Q_NPN_BEC
- R1, R10, R11, R2, R3, R4, R5, R6, R7, R8, R9: symbol Device:R_Small -> Device:R_Small_US
Connections:
- net 3.3V: now also D2.1 (VDD); no longer D2.4 (VDD)
- net DTR: now also Q2.2 (E); no longer Q2.3 (E)
- net EN: now also Q1.3 (C); no longer Q1.2 (C)
- net ESP_GND: now also D2.3 (VSS); no longer D2.2 (VSS)
- net GPIO0_BOOT: now also Q2.3 (C); no longer Q2.2 (C)
- net GPIO38: now also D2.4 (DIN); no longer D2.3 (DIN)
- net LED_OUT: now also D2.2 (DOUT); no longer D2.1 (DOUT)
- net RTS: now also Q1.2 (E); no longer Q1.3 (E)
Other:
- note added: "ESD Protection"

Commit message: silkscreen
Changed lines of the file:
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@@
 	(text "RTC CLOCK"
 		(exclude_from_sim no)
-		(at 175.26 89.408 0)
+		(at 166.878 89.154 0)
 		(effects
 			(font

Commit message: a little bit of a reorg
Parts:
- U3: symbol ESP32-S3-Breakout:ESP32-S3-WROOM -> RF_Module:ESP32-S3-WROOM-1
Other:
- moved on the sheet: C1, C3

Commit message: i think its ready for reddit.
Parts:
- FB1: value 500mA -> 1.5A; footprint Fuse:Fuse_0603_1608Metric -> Fuse:Fuse_1206_3216Metric; LCSC C69679 -> C2760275
- R3: value 1k -> 5.1k
Other:
- note added: "USB CHIPS AUTO POWER SWITCH"
- note removed: "USB POWER SWITCH"
- moved on the sheet: U6
Changed lines of the file:
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@@
 		)
 	)
-	(text "USB POWER SWITCH"
+	(text "USB CHIPS AUTO POWER SWITCH"
 		(exclude_from_sim no)
-		(at 29.718 166.624 0)
+		(at 14.224 166.116 0)
 		(effects
 			(font
@@
 				(bold yes)
 			)
+			(justify left)
 		)
 	)
 	(text "ESD Protection"
 		(exclude_from_sim no)
-		(at 86.614 55.626 0)
+		(at 73.406 55.626 0)
 		(effects
 			(font
@@
 	)
 	(junction
+		(at 46.99 191.77)
+		(diameter 0)
+		(color 0 0 0 0)
+	)
+	(junction
 		(at 185.42 110.49)
 		(diameter 0)
@@
 	(wire
 		(pts
-			(xy 110.49 187.96) (xy 110.49 190.5)
+			(xy 110.49 187.96) (xy 110.49 191.77)
 		)
 		(stroke
@@
 	(wire
 		(pts
-			(xy 86.36 76.2) (xy 86.36 74.93)
+			(xy 73.66 76.2) (xy 73.66 74.93)
 		)
 		(stroke
@@
 	(wire
 		(pts
-			(xy 86.36 59.69) (xy 86.36 62.23)
+			(xy 73.66 59.69) (xy 73.66 62.23)
 		)
 		(stroke
@@
 	(wire
 		(pts
+			(xy 46.99 191.77) (xy 54.61 191.77)
+		)
+		(stroke
+			(width 0)
+			(type default)
+		)
+	)
+	(wire
+		(pts
 			(xy 123.19 68.58) (xy 130.81 68.58)
 		)
@@
 	)
 	(label "USB_D+"
-		(at 91.44 67.31 0)
+		(at 68.58 67.31 180)
 		(fields_autoplaced yes)
 		(effects
@@
 				(size 1.27 1.27)
 			)
-			(justify left bottom)
+			(justify right bottom)
 		)
 		(property "Netclass" "DP_90R"
-			(at 91.44 68.58 0)
+			(at 68.58 68.58 0)
 			(effects
 				(font
@@
 					(italic yes)
 				)
-				(justify left)
+				(justify right)
 				(hide yes)
 			)
@@
 	)
 	(label "USB_D-"
-		(at 91.44 69.85 0)
+		(at 68.58 69.85 180)
 		(fields_autoplaced yes)
 		(effects
@@
 				(size 1.27 1.27)
 			)
-			(justify left bottom)
+			(justify right bottom)
 		)
 		(property "Netclass" "DP_90R"
-			(at 91.44 71.12 0)
+			(at 68.58 71.12 0)
 			(effects
 				(font
@@
 					(italic yes)
 				)
-				(justify left)
+				(justify right)
 				(hide yes)
 			)
@@
 	)
 	(label "HUB_D+"
-		(at 81.28 67.31 180)
+		(at 78.74 67.31 0)
 		(fields_autoplaced yes)
 		(effects
@@
 				(size 1.27 1.27)
 			)
-			(justify right bottom)
+			(justify left bottom)
 		)
 		(property "Netclass" "DP_90R"
-			(at 81.28 68.58 0)
+			(at 78.74 68.58 0)
 			(effects
 				(font
@@
 					(italic yes)
 				)
-				(justify right)
+				(justify left)
 				(hide yes)
 			)
@@
 	(label "VBUS"
 		(at 44.45 33.02 0)
+		(fields_autoplaced yes)
 		(effects
 			(font
@@
 			(justify left bottom)
 		)
+		(property "Netclass" "VBUS"
+			(at 44.45 34.29 0)
+			(effects
+				(font
+					(size 1.27 1.27)
+					(italic yes)
+				)
+				(justify left)
+			)
+		)
 	)
 	(label "UART_D+"
@@
 	)
 	(label "HUB_D-"
-		(at 81.28 69.85 180)
+		(at 78.74 69.85 0)
 		(fields_autoplaced yes)
 		(effects
@@
 				(size 1.27 1.27)
 			)
-			(justify right bottom)
+			(justify left bottom)
 		)
 		(property "Netclass" "DP_90R"
-			(at 81.28 71.12 0)
+			(at 78.74 71.12 0)
 			(effects
 				(font
@@
 					(italic yes)
 				)
-				(justify right)
+				(justify left)
 				(hide yes)
 			)
@@
 	)
 	(label "VBUS"
-		(at 86.36 59.69 180)
+		(at 73.66 59.69 0)
 		(effects
 			(font
 				(size 1.27 1.27)
 			)
-			(justify right bottom)
+			(justify left bottom)
 		)
 	)
@@
 	(hierarchical_label "ESP_GND"
 		(shape input)
-		(at 86.36 76.2 180)
+		(at 73.66 76.2 0)
 		(effects
 			(font
 				(size 1.27 1.27)
 			)
-			(justify right)
+			(justify left)
 		)
 	)
@@
 	(hierarchical_label "ESP_GND"
 		(shape input)
-		(at 46.99 191.77 0)
+		(at 54.61 191.77 0)
 		(effects
 			(font
@@
 	(hierarchical_label "ESP_GND"
 		(shape input)
-		(at 110.49 190.5 0)
+		(at 110.49 191.77 0)
 		(effects
 			(font
@@
 			)
 		)
-		(property "Value" "1k"
+		(property "Value" "5.1k"
 			(at 176.022 172.72 90)
 			(effects
@@
 		(lib_name "USBLC6-2SC6_1")
 		(lib_id "Power_Protection:USBLC6-2SC6")
-		(at 86.36 67.31 0)
+		(at 73.66 67.31 0)
+		(mirror y)
 		(unit 1)
 		(exclude_from_sim no)
@@
 		(fields_autoplaced yes)
 		(property "Reference" "U6"
-			(at 88.0111 59.69 0)
+			(at 72.0089 59.69 0)
 			(effects
 				(font
@@
 		)
 		(property "Value" "USBLC6-2SC6"
-			(at 88.0111 62.23 0)
+			(at 72.0089 62.23 0)
 			(effects
 				(font
@@
 		)
 		(property "Footprint" "Package_TO_SOT_SMD:SOT-23-6"
-			(at 87.63 73.66 0)
+			(at 72.39 73.66 0)
 			(effects
 				(font
@@
 		)
 		(property "Datasheet" "https://www.st.com/resource/en/datasheet/usblc6-2.pdf"
-			(at 87.63 75.565 0)
+			(at 72.39 75.565 0)
 			(effects
 				(font
@@
 		)
 		(property "Description" "Very low capacitance ESD protection diode, 2 data-line, SOT-23-6"
-			(at 86.36 67.31 0)
+			(at 73.66 67.31 0)
 			(effects
 				(font
@@
 		)
 		(property "LCSC" "C7519"
-			(at 86.36 67.31 0)
+			(at 73.66 67.31 0)
 			(effects
 				(font
@@
 			)
 		)
-		(property "Value" "500mA"
+		(property "Value" "1.5A"
 			(at 69.8119 29.21 90)
 			(effects
@@
 			)
 		)
-		(property "Footprint" "Fuse:Fuse_0603_1608Metric"
+		(property "Footprint" "Fuse:Fuse_1206_3216Metric"
 			(at 69.85 34.798 90)
 			(effects
@@
 			)
 		)
-		(property "LCSC" "C69679"
+		(property "LCSC" "C2760275"
 			(at 69.85 33.02 90)
 			(effects

Commit message: another full pass over the schematic and layout
Parts:
- R1, R2: LCSC C105580 -> (none)
Other:
- note added: "USB CHIPS POWER SAVER"
- note removed: "USB CHIPS AUTO POWER SWITCH"
- title: (none) -> https://github.com/hoeken/ESP32-S3-Template
- moved on the sheet: C1, C3, C6, C7, U3

Commit message: pulled in brineomatic version
Parts:
- D1: LCSC (none) -> C191023
- D2: renamed from D3; value LED -> RED; LCSC (none) -> C965799
- J3: renamed from J1; Position Offset (none) -> 0.0,1.27
- Q1: renamed from Q3; LCSC (none) -> C112086
- R1: renamed from R11; value 100 -> 100R
- SW1, SW2: footprint Button_Switch_SMD:SW_SPST_B3U-1000P -> Button_Switch_THT:SW_Tactile_SPST_Angled_PTS645Vx58-2LFS; LCSC C843684 -> C557599; Rotation Offset (none) -> 180
- U1: renamed from U3; footprint RF_Module:ESP32-S3-WROOM-1 -> yarrboard:ESP32-S3-WROOM-1; LCSC (none) -> C2913202; Position Offset (none) -> 0,-3.6195
- U2: renamed from U6; Rotation Offset (none) -> 90
- U3: renamed from U5; LCSC (none) -> C424705
- U4: renamed from U2; footprint Package_DFN_QFN:QFN-24-1EP_4x4mm_P0.5mm_EP2.7x2.7mm_ThermalVias -> yarrboard:QFN-24-1EP_4x4mm_P0.5mm_EP2.7x2.7mm_ThermalVias; LCSC (none) -> C5187527; Rotation Offset (none) -> 180
- U5: renamed from U1; footprint Package_DFN_QFN:QFN-16-1EP_3x3mm_P0.5mm_EP1.7x1.7mm_ThermalVias -> yarrboard:QFN-16-1EP_3x3mm_P0.5mm_EP1.7x1.7mm_ThermalVias; LCSC (none) -> C2846043; Rotation Offset (none) -> 180
- renumbered C12 to C10, C5 to C11, C2 to C12, C4 to C13, C15 to C14, C16 to C15, C14 to C16, C10 to C18, C11 to C19, C3 to C2, C13 to C3, C8 to C4, C18 to C5, C9 to C8, C19 to C9, D2 to D3, Q1 to Q2, Q2 to Q3, R5 to R10, R4 to R11, R9 to R2, R10 to R3, R1 to R4, R2 to R5, R3 to R6, R8 to R7, R6 to R8, R7 to R9, Y2 to Y1, Y1 to Y2
Connections:
- net 3.3V: now also D2.2 (A); no longer R6.1
- net ESP_GND: now also R6.2; no longer D2.1 (K)
- new net: D2.1 (K), R6.1
Other:
- note added: "POWER"
- note removed: "POWER LED"
- moved on the sheet: D2, R6
